File: zlvdt_pcb/zlvdt_pcb.kicad_pcb (KiCad board)
At the start: 2 copper layers, 27.9 x 68.6 mm, 10 parts, among them J1 ESP_02x03_Female, J2 LVDT_conn, U1 LM358

Commit message: Плата переразведена топором
Parts:
- moved R5 5.24 mm to (113.0, 81.3), turned to -90 degrees
Routing:
- net GND: track 45.0 -> 35.7 mm
- net Net-(D1-Pad2): track 15.1 -> 22.5 mm
- net esp_16_adc2_ch5_lvdt: track 20.0 -> 13.1 mm
- net esp_15_adc2_ch4_exc: track 40.2 -> 37.8 mm
- net Net-(D1-Pad1): track 14.7 -> 13.5 mm
- net Net-(R1-Pad2): track 23.3 -> 22.3 mm

Commit message: test version
Parts:
- removed D1: PMEG1030EJ, Diode_SMD:D_SMA_Handsoldering
- R4: value 10k -> 33k
Routing:
- net esp_15_adc2_ch4_exc: track 37.8 -> 0.00 mm
- net GND: track 35.7 -> 0.00 mm
- net Net-(R3-Pad2): track 22.5 -> 0.00 mm
- net Net-(R1-Pad2): track 22.3 -> 0.00 mm
- net Net-(D2-Pad2): track 13.5 -> 0.00 mm
- net lvdt_input: track 13.2 -> 0.00 mm
- net esp_16_adc2_ch5_lvdt: track 13.1 -> 0.00 mm
- net +5V: track 5.07 -> 0.00 mm
- net esp_17_dac1: track 1.63 -> 0.00 mm
