File: zlvdt_pcb/zlvdt_pcb.kicad_sch (KiCad schematic)
At the start: 10 parts, among them J1 ESP_02x03_Female, J2 LVDT_conn, U1 LM358

Commit message: test version
Parts:
- removed D1: PMEG1030EJ, Diode_SMD:D_SMA_Handsoldering, symbol Diode:PMEG1030EJ
Changed lines of the file:
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@@
 (kicad_sch (version 20211123) (generator eeschema)
   (paper "A4")
-  (junction (at 92.71 44.45) (diameter 0) (color 0 0 0 0)
-  )
   (junction (at 92.71 39.37) (diameter 0) (color 0 0 0 0)
   )
-  (junction (at 109.22 36.83) (diameter 0) (color 0 0 0 0)
-  )
   (junction (at 119.38 36.83) (diameter 0) (color 0 0 0 0)
   )
@@
     (stroke (width 0) (type default) (color 0 0 0 0))
   )
-  (wire (pts (xy 101.6 44.45) (xy 92.71 44.45))
-    (stroke (width 0) (type default) (color 0 0 0 0))
-  )
   (wire (pts (xy 55.88 58.42) (xy 53.34 58.42))
     (stroke (width 0) (type default) (color 0 0 0 0))
@@
     (stroke (width 0) (type default) (color 0 0 0 0))
   )
-  (wire (pts (xy 92.71 44.45) (xy 92.71 39.37))
+  (wire (pts (xy 92.71 39.37) (xy 92.71 52.07))
     (stroke (width 0) (type default) (color 0 0 0 0))
   )
@@
     (stroke (width 0) (type default) (color 0 0 0 0))
   )
-  (wire (pts (xy 109.22 44.45) (xy 109.22 36.83))
-    (stroke (width 0) (type default) (color 0 0 0 0))
-  )
   (wire (pts (xy 157.48 54.61) (xy 160.02 54.61))
-    (stroke (width 0) (type default) (color 0 0 0 0))
-  )
-  (wire (pts (xy 92.71 44.45) (xy 92.71 52.07))
     (stroke (width 0) (type default) (color 0 0 0 0))
   )
@@
     (pin "2")
   )
-  (symbol (lib_id "Diode:PMEG1030EJ") (at 105.41 44.45 180) (unit 1)
-    (in_bom yes) (on_board yes) (fields_autoplaced)
-    (property "Reference" "D1" (id 0) (at 105.7275 39.5056 0))
-    (property "Value" "PMEG1030EJ" (id 1) (at 105.7275 42.0425 0))
-    (property "Footprint" "Diode_SMD:D_SMA_Handsoldering" (id 2) (at 105.41 40.005 0)
-      (effects (font (size 1.27 1.27)) hide)
-    )
-    (property "Datasheet" "https://assets.nexperia.com/documents/data-sheet/PMEG1030EH_EJ.pdf" (id 3) (at 105.41 44.45 0)
-      (effects (font (size 1.27 1.27)) hide)
-    )
-    (pin "1")
-    (pin "2")
-  )
   (symbol (lib_id "power:GND") (at 93.98 27.94 180) (unit 1)
     (in_bom yes) (on_board yes) (fields_autoplaced)
@@
       (reference "#PWR0109") (unit 1) (value "GND") (footprint "")
     )
-    (path "/85152557-41b7-41cb-9451-0573f390a97d"
-      (reference "D1") (unit 1) (value "PMEG1030EJ") (footprint "Diode_SMD:D_SMA_Handsoldering")
-    )
     (path "/e242af74-9cf3-4dc6-ad10-9a9b65931d09"
